File: HW_ESP32S3_Template/HW_ESP32S3_Template.kicad_sch (KiCad schematic)
At the start: 32 parts, among them J1 Conn_02x03_Odd_Even, Q1 BSN20, Q2 BSN20, Q3 BSN20, SW1 K2-1102SP-C4SC-04, SW2 K2-1102SP-C4SC-04, U1 ESP32-S3-WROOM-1(N8R2), U2 S4B-PH-SM4-K-TB(LF)(SN), U3 LD1117S33TR

Commit message: set programming connector to 'not on BOM'
Parts:
- J1: now left out of the parts list
Changed lines of the file:
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@@
   )
   (symbol (lib_id "Connector_Generic:Conn_02x03_Odd_Even") (at 68.58 22.225 0) (unit 1)
-    (in_bom yes) (on_board yes) (dnp no) (fields_autoplaced)
+    (in_bom no) (on_board yes) (dnp no) (fields_autoplaced)
     (property "Reference" "J1" (at 69.85 14.605 0)
       (effects (font (size 1.27 1.27)))
